Commit message: 类似于b2w的碰撞体

File: nezha_description/urdf/nezha_description.urdf (robot description, URDF)
Before this commit: robot nezha_description, 18 links, 17 joints
Links:
- added link downboard_link; collision box size=0.11 0.10 0.009
- added link lidar_link; collision box size=0.11 0.10 0.15
- added link upboard_link; collision box size=0.11 0.10 0.009
- link FL_calf_Link: geometry collision mesh filename=package://nezha_description/meshes/FL_calf_Link.STL; visual mesh filename=package://nezha_description/meshes/FL_calf_Link.STL
- link FL_foot: geometry collision mesh filename=package://nezha_description/meshes/FL_foot_Link.STL; visual mesh filename=package://nezha_description/meshes/FL_foot_Link.STL
- link FL_hip_Link: geometry collision cylinder length=0.165 radius=0.0625; visual mesh filename=package://nezha_description/meshes/FL_hip_Link.STL
- link FL_thigh_Link: geometry collision box size=0.120 0.050 0.320; visual mesh filename=package://nezha_description/meshes/FL_thigh_Link.STL
- link FR_calf_Link: geometry collision mesh filename=package://nezha_description/meshes/FR_calf_Link.STL; visual mesh filename=package://nezha_description/meshes/FR_calf_Link.STL
- link FR_foot: geometry collision mesh filename=package://nezha_description/meshes/FR_foot_Link.STL; visual mesh filename=package://nezha_description/meshes/FR_foot_Link.STL
- link FR_hip_Link: geometry collision cylinder length=0.165 radius=0.0625; visual mesh filename=package://nezha_description/meshes/FR_hip_Link.STL
- link FR_thigh_Link: geometry collision box size=0.120 0.050 0.320; visual mesh filename=package://nezha_description/meshes/FR_thigh_Link.STL
- link RL_calf_Link: geometry collision mesh filename=package://nezha_description/meshes/RL_calf_Link.STL; visual mesh filename=package://nezha_description/meshes/RL_calf_Link.STL
- link RL_foot: geometry collision mesh filename=package://nezha_description/meshes/RL_foot_Link.STL; visual mesh filename=package://nezha_description/meshes/RL_foot_Link.STL
- link RL_hip_Link: geometry collision cylinder length=0.165 radius=0.0625; visual mesh filename=package://nezha_description/meshes/RL_hip_Link.STL
- link RL_thigh_Link: geometry collision box size=0.120 0.050 0.320; visual mesh filename=package://nezha_description/meshes/RL_thigh_Link.STL
- link RR_calf_Link: geometry collision mesh filename=package://nezha_description/meshes/RR_calf_Link.STL; visual mesh filename=package://nezha_description/meshes/RR_calf_Link.STL
- link RR_foot: geometry collision mesh filename=package://nezha_description/meshes/RR_foot_Link.STL; visual mesh filename=package://nezha_description/meshes/RR_foot_Link.STL
- link RR_hip_Link: geometry collision cylinder length=0.165 radius=0.0625; visual mesh filename=package://nezha_description/meshes/RR_hip_Link.STL
- link RR_thigh_Link: geometry collision box size=0.120 0.050 0.320; visual mesh filename=package://nezha_description/meshes/RR_thigh_Link.STL
- link trunk_link: geometry collision box size=0.710 0.380 0.190; visual mesh filename=package://nezha_description/meshes/trunk_link.STL
Joints:
- added joint downboard_joint: type fixed, parent trunk_link, child downboard_link, origin xyz=0.42 -0.0375 -0.105 rpy=0 0 0, axis 0 0 0
- added joint lidar_joint: type fixed, parent trunk_link, child lidar_link, origin xyz=0.55 -0.0375 0.07 rpy=0 0 0, axis 0 0 0
- added joint upboard_joint: type fixed, parent trunk_link, child upboard_link, origin xyz=0.42 -0.0375 0.085 rpy=0 0 0, axis 0 0 0

Commit message: 赵任宇去合肥后改的

File: nezha_description/urdf/nezha_description.urdf (robot description, URDF)
Before this commit: robot nezha_description, 18 links, 17 joints
Links:
- removed link FL_calf_Link
- removed link FL_hip_Link
- removed link FL_thigh_Link
- removed link FR_calf_Link
- removed link FR_hip_Link
- removed link FR_thigh_Link
- removed link RL_calf_Link
- removed link RL_hip_Link
- removed link RL_thigh_Link
- removed link RR_calf_Link
- removed link RR_hip_Link
- removed link RR_thigh_Link
- removed link imu_fixed_joint
- removed link trunk_link
- added link FL_calf, mass 1.39639981011161; collision box size=0.05 0.045 0.390; visual mesh filename=package://nezha_description/meshes/FL_calf_Link.STL
- added link FL_hip, mass 4.95777307433676; visual mesh filename=package://nezha_description/meshes/FL_hip_Link.STL
- added link FL_thigh, mass 1.98935336838793; visual mesh filename=package://nezha_description/meshes/FL_thigh_Link.STL
- added link FR_calf, mass 1.39639981011161; collision box size=0.05 0.045 0.390; visual mesh filename=package://nezha_description/meshes/FR_calf_Link.STL
- added link FR_hip, mass 4.95777307433546; visual mesh filename=package://nezha_description/meshes/FR_hip_Link.STL
- added link FR_thigh, mass 1.99301153063505; visual mesh filename=package://nezha_description/meshes/FR_thigh_Link.STL
- added link RL_calf, mass 1.39639981011242; collision box size=0.05 0.045 0.390; visual mesh filename=package://nezha_description/meshes/RL_calf_Link.STL
- added link RL_hip, mass 4.95777307433676; visual mesh filename=package://nezha_description/meshes/RL_hip_Link.STL
- added link RL_thigh, mass 1.99301153063505; visual mesh filename=package://nezha_description/meshes/RL_thigh_Link.STL
- added link RR_calf, mass 1.39639981011242; collision box size=0.05 0.045 0.390; visual mesh filename=package://nezha_description/meshes/RR_calf_Link.STL
- added link RR_hip, mass 4.95777307436896; visual mesh filename=package://nezha_description/meshes/RR_hip_Link.STL
- added link RR_thigh, mass 1.98935336838794; visual mesh filename=package://nezha_description/meshes/RR_thigh_Link.STL
- added link imu_fixed_link, mass 0.0406912140939172; visual mesh filename=package://nezha_description/meshes/imu_fixed_joint.STL
- added link trunk, mass 37.7952892364436; collision box size=1.121 0.400 0.230; visual mesh filename=package://nezha_description/meshes/trunk_link.STL
- link FL_foot: mass 8.83568216072149 -> 1.93478304677791
- link FR_foot: mass 8.835682161799 -> 1.93478304677791
- link RL_foot: mass 8.83568216072149 -> 1.93478304677792
- link RR_foot: mass 8.83568216072149 -> 1.93478304677791
Joints:
- joint FL_calf_joint: child FL_calf_Link -> FL_calf; limit lower=-2.478 upper=-0.768 effort=300 velocity=30 -> lower=-2.478 upper=-0.768 effort=160 velocity=30; origin xyz=0 0.0619999999999968 -0.330000000000104 rpy=0 0 0 -> xyz=0 0.061999999999997 -0.330000000000104 rpy=0 0 0; parent FL_thigh_Link -> FL_thigh
- joint FL_foot_joint: limit lower=-9999 upper=9999 effort=60 velocity=100 -> lower=-999999 upper=999999 effort=60 velocity=100; origin xyz=0 -0.0140000000000013 -0.329999999999984 rpy=0 0 0 -> xyz=0 -0.0165871612253468 -0.329999999999984 rpy=0 0 0; parent FL_calf_Link -> FL_calf
- joint FL_hip_joint: child FL_hip_Link -> FL_hip; limit lower=-0.7854 upper=1.5533 effort=300 velocity=30 -> lower=-0.7854 upper=1.5533 effort=160 velocity=30; origin xyz=0.347120192019755 0.0485117531253507 -0.0290000000000001 rpy=0 0 0 -> xyz=0.346 0.0849999999999999 -0.0290000000000001 rpy=0 0 0; parent trunk_link -> trunk
- joint FL_thigh_joint: child FL_thigh_Link -> FL_thigh; limit lower=-1.571 upper=1.571 effort=300 velocity=30 -> lower=-1.571 upper=2.7 effort=160 velocity=30; parent FL_hip_Link -> FL_hip
- joint FR_calf_joint: child FR_calf_Link -> FR_calf; limit lower=-2.478 upper=-0.768 effort=300 velocity=30 -> lower=-2.478 upper=-0.768 effort=160 velocity=30; origin xyz=0 -0.0619999999999982 -0.329999999999805 rpy=0 0 0 -> xyz=0 -0.061999999999997 -0.330000000000104 rpy=0 0 0; parent FR_thigh_Link -> FR_thigh
- joint FR_foot_joint: limit lower=-9999 upper=9999 effort=60 velocity=100 -> lower=-999999 upper=999999 effort=60 velocity=100; origin xyz=0 0.0191743224506925 -0.329999999987678 rpy=0 0 0 -> xyz=0 0.0165871612253468 -0.329999999999984 rpy=0 0 0; parent FR_calf_Link -> FR_calf
- joint FR_hip_joint: child FR_hip_Link -> FR_hip; limit lower=-1.5533 upper=0.7854 effort=300 velocity=30 -> lower=-1.5533 upper=0.7854 effort=160 velocity=30; origin xyz=0.34712 -0.12149 -0.029 rpy=0 0 0 -> xyz=0.346 -0.0849999999999999 -0.0290000000000001 rpy=0 0 0; parent trunk_link -> trunk
- joint FR_thigh_joint: child FR_thigh_Link -> FR_thigh; limit lower=-1.571 upper=1.571 effort=300 velocity=30 -> lower=-1.571 upper=2.7 effort=160 velocity=30; parent FR_hip_Link -> FR_hip
- joint RL_calf_joint: child RL_calf_Link -> RL_calf; limit lower=0.768 upper=2.478 effort=300 velocity=30 -> lower=0.768 upper=2.478 effort=160 velocity=30; origin xyz=0 0.0619999999999982 -0.329999999987498 rpy=0 0 0 -> xyz=0 0.061999999999997 -0.330000000000104 rpy=0 0 0; parent RL_thigh_Link -> RL_thigh
- joint RL_foot_joint: limit lower=-9999 upper=9999 effort=60 velocity=100 -> lower=-999999 upper=999999 effort=60 velocity=100; origin xyz=0 -0.0191743224506925 -0.329999999999986 rpy=0 0 0 -> xyz=0 -0.0165871612253468 -0.329999999999984 rpy=0 0 0; parent RL_calf_Link -> RL_calf
- joint RL_hip_joint: child RL_hip_Link -> RL_hip; limit lower=-0.7854 upper=1.5533 effort=300 velocity=30 -> lower=-0.7854 upper=1.5533 effort=160 velocity=30; origin xyz=-0.34488 0.048512 -0.029 rpy=0 0 0 -> xyz=-0.346 0.0849999999999999 -0.0290000000000001 rpy=0 0 0; parent trunk_link -> trunk
- joint RL_thigh_joint: child RL_thigh_Link -> RL_thigh; limit lower=-1.571 upper=1.571 effort=300 velocity=30 -> lower=-2.7 upper=1.571 effort=160 velocity=30; parent RL_hip_Link -> RL_hip
- joint RR_calf_joint: child RR_calf_Link -> RR_calf; limit lower=0.768 upper=2.478 effort=300 velocity=30 -> lower=0.768 upper=2.478 effort=160 velocity=30; origin xyz=0 -0.0619999999999969 -0.329999999460342 rpy=0 0 0 -> xyz=0 -0.061999999999997 -0.330000000000104 rpy=0 0 0; parent RR_thigh_Link -> RR_thigh
- joint RR_foot_joint: limit lower=-9999 upper=9999 effort=60 velocity=100 -> lower=-999999 upper=999999 effort=60 velocity=100; origin xyz=0 0.0140000000000008 -0.329999999987677 rpy=0 0 0 -> xyz=0 0.0165871612253468 -0.329999999999984 rpy=0 0 0; parent RR_calf_Link -> RR_calf
- joint RR_hip_joint: child RR_hip_Link -> RR_hip; limit lower=-1.5533 upper=0.7854 effort=300 velocity=30 -> lower=-1.5533 upper=0.7854 effort=160 velocity=30; origin xyz=-0.344879807980245 -0.121488246874649 -0.0290000000000001 rpy=0 0 0 -> xyz=-0.346 -0.0849999999999999 -0.0290000000000001 rpy=0 0 0; parent trunk_link -> trunk
- joint RR_thigh_joint: child RR_thigh_Link -> RR_thigh; limit lower=-1.571 upper=1.571 effort=300 velocity=30 -> lower=-2.7 upper=1.571 effort=160 velocity=30; parent RR_hip_Link -> RR_hip
- joint imu_fixed_joint: child imu_fixed_joint -> imu_fixed_link; parent trunk_link -> trunk
